File: Project SBO - Autogenerated Samoklava/board.kicad_pcb (KiCad board)
At the start: 2 copper layers, 122.3 x 118.1 mm, 44 parts, among them J1 Jumper, J2 Jumper

Commit message: who knows
Parts:
- added D10: , ComboDiode, F.Cu at (36.0, -27.3)
- added D14: , ComboDiode, F.Cu at (54.0, -23.9)
- added D18: , ComboDiode, F.Cu at (72.0, -22.2)
- added D2: , ComboDiode, F.Cu at (0.00, -12.0)
- added D22: , ComboDiode, F.Cu at (80.9, 21.4)
- added D6: , ComboDiode, F.Cu at (18.0, -23.9)
- added G***: LOGO, Track:pivot_hat_smoll, F.Cu at (37.8, 4.20)
- added G***: LOGO, Track:jammer_hat_2_smol, F.Cu at (36.7, 2.97)
- added S10: , PG1350, F.Cu at (36.0, -32.3)
- added S14: , PG1350, F.Cu at (54.0, -28.9)
- added S18: , PG1350, F.Cu at (72.0, -27.2)
- added S2: , PG1350, F.Cu at (0.00, -17.0)
- added S22: , PG1350, F.Cu at (83.4, 17.1)
- added S6: , PG1350, F.Cu at (18.0, -28.9)
- moved S11 17.0 mm to (36.0, -49.3)
- moved D11 17.0 mm to (36.0, -44.3)
Routing:
- net row_home: track 0.00 -> 118.5 mm
- net home_thumb: track 0.00 -> 29.3 mm
- net index_home: track 0.00 -> 29.1 mm
- net middle_home: track 0.00 -> 29.1 mm
- net pinky_home: track 0.00 -> 29.1 mm
- net ring_home: track 0.00 -> 29.1 mm
- net inner_home: track 0.00 -> 29.0 mm
- net col_inner: track 227.6 -> 255.7 mm
- net row_thumb: track 71.3 -> 98.9 mm
- net middle_top: track 55.2 -> 29.1 mm
- net col_index: track 204.9 -> 230.7 mm
- net row_top: track 145.7 -> 121.2 mm
- net col_middle: track 227.3 -> 238.7 mm
- net col_ring: track 193.6 -> 203.1 mm
- net row_extra: track 141.5 -> 150.6 mm
Other:
- board text added: "Project SBO Schism samoklava remix Kel to Pay 2024 kel.to.pay@gmail.com"
- board text removed: "samoklava v0.3 by soundmonster"
